File: Drone Launcher PCB/Drone Launcher PCB.kicad_pcb (KiCad board)
At the start: 4 copper layers, 65 x 30 mm, 55 parts, among them Q7 AO3407A, SW1 MSK12C02, U1 BQ24075RGTR, U12 AP2112K-3.3, U2 ZX-PH2.0-WT2P, U3 TPS61023DRLR, U4 DW03C_C41367942, U6 ESP32-C3-MINI-1U-N4

Commit message: sync
Parts:
- added G***: LOGO, LOGO, F.Cu at (38.9, 43.4)
- moved R24 3.93 mm to (31.2, 28.5), turned to 0 degrees
- moved R36 3.66 mm to (19.5, 16.8)
- moved LED5 2.93 mm to (42.0, 28.6)
- moved R12 2.38 mm to (32.0, 22.8), turned to 180 degrees
- moved R29 2.23 mm to (38.7, 28.6), turned to 0 degrees
- moved R11 2.16 mm to (33.8, 17.6), turned to 180 degrees
- moved R18 1.63 mm to (3.70, 22.4), turned to 0 degrees
- moved D5 1.59 mm to (22.4, 19.2)
- moved R34 1.50 mm to (25.0, 21.9)
- moved C32 1.44 mm to (31.2, 18.7)
- moved R38 1.30 mm to (62.6, 12.3), turned to 0 degrees
- moved R37 1.17 mm to (20.1, 22.1)
- moved U1 1.15 mm to (35.6, 20.6)
- moved C40 1.15 mm to (39.2, 21.4)
- moved C41 1.15 mm to (39.2, 23.1)
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Routing:
- net GND: track 13.9 -> 112.9 mm, vias 8 -> 58
- net ESP32_VMON_ADC: track 0.00 -> 50.2 mm, vias 0 -> 2
- net Net-(U6-EN): track 0.00 -> 31.6 mm, vias 0 -> 2
- net BATT_SW+: track 5.33 -> 34.5 mm, vias 0 -> 2
- net BATT+: track 0.00 -> 26.0 mm
- net USB_VBUS: track 0.00 -> 24.8 mm
- net Net-(Q7-G): track 0.00 -> 21.7 mm, vias 0 -> 2
- net Net-(C27-Pad2): track 0.00 -> 18.6 mm
- net Net-(U6-IO9): track 0.00 -> 16.8 mm, vias 0 -> 2
- net BATT_OUT: track 0.00 -> 16.4 mm
- net +5V: track 0.00 -> 14.5 mm
- net Net-(LED5-K): track 0.00 -> 12.5 mm, vias 0 -> 2
- net Net-(LED6-K): track 0.00 -> 11.8 mm, vias 0 -> 2
- net Net-(U6-RXD0): track 0.00 -> 9.60 mm
- net +3.3V: track 0.00 -> 9.32 mm, vias 0 -> 8
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- added copper zone on In2.Cu, net +3.3V
- added copper zone on In1.Cu, net GND
Other:
- board text added: "CHRG"
- board text added: "OFF"
- board text added: "ON"
- board text added: "PG"
